File: Hardware/Kicad/TRH9000/TRH9000.kicad_pcb (KiCad board)
At the start: 4 copper layers, 99.1 x 63.5 mm, 65 parts, among them J1 RGB, Q1 BC817, U1 V9990, U2 KM428C256, U3 KM428C256, U4 74HC138, U6 LMH1980, U7 74HC32, X1 14.31818MHz, Y1 21.47727Mhz

Commit message: Prototype board. Fixes to the main project. Readme updates.
Parts:
- removed REF**: OSHW-Logo_11.4x12mm_SilkScreen, Symbol:OSHW-Logo_11.4x12mm_SilkScreen
- removed RV1-R, RV2-G, RV3-B: 500R, Potentiometer_SMD:Potentiometer_Bourns_3314G_Vertical
- added RV1: 500R, Potentiometer_SMD:Potentiometer_Bourns_3314G_Vertical, B.Cu at (146.9, 87.1)
- added RV2: 500R, Potentiometer_SMD:Potentiometer_Bourns_3314G_Vertical, B.Cu at (152.9, 87.1)
- added RV3: 500R, Potentiometer_SMD:Potentiometer_Bourns_3314G_Vertical, B.Cu at (158.9, 87.0)
Connections:
- U2 pad 12: GND -> /VDP/~{V1_WE}
- U2 pad 13: /VDP/~{V1_WE} -> unconnected-(U2-Pad13)
- U2 pad 21: GND -> unconnected-(U2-Pad21)
- U3 pad 12: GND -> /VDP/~{V0_WE}
- U3 pad 13: /VDP/~{V0_WE} -> unconnected-(U3-Pad13)
- U3 pad 21: GND -> unconnected-(U3-Pad21)
Routing:
- net GND: track 147.6 -> 135.9 mm, vias 37 -> 33
- net /VDP/~{V1_WE}: track 29.5 -> 28.2 mm
- net /VDP/~{V0_WE}: track 43.5 -> 44.6 mm

Commit message: Updates during tests with prototype
Connections:
- U4 pad 9: Net-(U4-Pad9) -> Net-(U7-Pad12)
- U7 pad 11: unconnected-(U7-Pad11) -> /~{BUSDIR}
- U7 pad 12: unconnected-(U7-Pad12) -> Net-(U7-Pad12)
- U7 pad 13: unconnected-(U7-Pad13) -> /~{RD}
- U7 pad 2: Net-(U4-Pad9) -> Net-(U7-Pad12)
- U7 pad 5: Net-(U4-Pad9) -> Net-(U7-Pad12)
Routing:
- net /~{BUSDIR}: track 0.00 -> 38.6 mm, vias 0 -> 1
- net Net-(U7-Pad12): track 0.00 -> 20.2 mm, vias 0 -> 2
- net Net-(U4-Pad9): track 14.8 -> 0.00 mm, vias 2 -> 0
- net /~{RD}: track 25.5 -> 30.8 mm
- net GNDA: track 116.9 -> 119.2 mm
- net /VDP/~{VDPR}: track 45.7 -> 44.8 mm
