File: Hardware/Kicad/TRH9000/TRH9000_VDP.kicad_sch (KiCad schematic)
At the start: 13 parts, among them U1 V9990, U2 KM428C256, U3 KM428C256, X1 14.31818MHz, Y1 21.47727Mhz

Commit message: Prototype board. Fixes to the main project. Readme updates.
Connections:
- net ~{V0_WE}: now also U3.12 (~{WB}/~{WE}); no longer U3.13 (R~{WB}/~{WE})
- net ~{V1_WE}: now also U2.12 (~{WB}/~{WE}); no longer U2.13 (R~{WB}/~{WE})
Changed lines of the file:
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@@
     )
     (property "Value" "KM428C256" (id 1) (at 266.7 106.68 0))
-    (property "Footprint" "trh9000:SOJ-40_400mil" (id 2) (at 273.05 85.09 0)
+    (property "Footprint" "trh9000:SOJ-40_400mil" (id 2) (at 288.29 111.76 0)
       (effects (font (size 1.27 1.27)) hide)
     )
-    (property "Datasheet" "https://pdf1.alldatasheet.com/datasheet-pdf/view/129863/SAMSUNG/KM428C256.html" (id 3) (at 273.05 85.09 0)
+    (property "Datasheet" "https://pdf1.alldatasheet.com/datasheet-pdf/view/129863/SAMSUNG/KM428C256.html" (id 3) (at 273.05 114.3 0)
       (effects (font (size 1.27 1.27)) hide)
     )
@@
     (pin "10")
     (pin "11")
-    (pin "13")
+    (pin "12")
     (pin "14")
     (pin "15")
@@
     (pin "9")
     (pin "1")
-    (pin "12")
+    (pin "13")
     (pin "20")
     (pin "21")
@@
     (pin "2")
   )
-  (symbol (lib_name "KM428C256_1") (lib_id "TRH9000:KM428C256") (at 275.59 173.99 0) (unit 1)
+  (symbol (lib_id "TRH9000:KM428C256") (at 275.59 173.99 0) (unit 1)
     (in_bom yes) (on_board yes)
     (property "Reference" "U2" (id 0) (at 265.43 149.86 0)
@@
     )
     (property "Value" "KM428C256" (id 1) (at 269.24 205.74 0))
-    (property "Footprint" "trh9000:SOJ-40_400mil" (id 2) (at 275.59 184.15 0)
+    (property "Footprint" "trh9000:SOJ-40_400mil" (id 2) (at 290.83 210.82 0)
       (effects (font (size 1.27 1.27)) hide)
     )
-    (property "Datasheet" "https://pdf1.alldatasheet.com/datasheet-pdf/view/129863/SAMSUNG/KM428C256.html" (id 3) (at 275.59 184.15 0)
+    (property "Datasheet" "https://pdf1.alldatasheet.com/datasheet-pdf/view/129863/SAMSUNG/KM428C256.html" (id 3) (at 275.59 213.36 0)
       (effects (font (size 1.27 1.27)) hide)
     )
@@
     (pin "10")
     (pin "11")
-    (pin "13")
+    (pin "12")
     (pin "14")
     (pin "15")
@@
     (pin "9")
     (pin "1")
-    (pin "12")
+    (pin "13")
     (pin "20")
     (pin "21")

Commit message: Multiple changes. Check the dev log.
Parts:
- renumbered C1 to C3, R5 to R1, R3 to R2, R6 to R3, R1 to R5, R2 to R6, U1 to U3, U3 to U4, U2 to U5
Connections:
- net ~{VDPR}: now also U3.3 (~{CSR}); no longer U3.2 (~{CSW})
- net ~{VDPW}: now also U3.2 (~{CSW}); no longer U3.3 (~{CSR})

Commit message: Multiple changes.
Connections:
- net ~{V0_WE}: now also U4.13 (~{WB}/~{WE}); no longer U4.12 (~{WB}/~{WE})
- net ~{V1_WE}: now also U5.13 (~{WB}/~{WE}); no longer U5.12 (~{WB}/~{WE})
Other:
- note removed: "VGA clocks: ------------- 640x400 (70Hz) - 25.175 MHz 640x480 (60Hz) - 25.175 MHz Pal clocks: ------------- 704x576 (50Hz) - 4.43361875 MHz NTSC clocks: -------------- 704x480 (60Hz) - 3.579545 MHz"
