File: Hardware/Kicad/TRH9000/TRH9000.kicad_sch (KiCad schematic)
At the start: 10 parts, among them U4 74HC138, U7 74HC32

Commit message: Routing, readme, etc
Parts:
- C11, C12, C25, C26: now left out of the parts list
Changed lines of the file:
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@@
   )
   (symbol (lib_id "LRJ-parts:C_CL21B105KBFNNNF") (at 66.04 100.33 90) (unit 1)
-    (in_bom yes) (on_board yes)
+    (in_bom no) (on_board no)
     (property "Reference" "C25" (id 0) (at 62.23 99.06 90)
       (effects (font (size 1.143 1.143)))
@@
   )
   (symbol (lib_id "LRJ-parts:C_CC0805JPX7R9BB104") (at 72.39 116.84 90) (unit 1)
-    (in_bom yes) (on_board yes)
+    (in_bom no) (on_board no)
     (property "Reference" "C12" (id 0) (at 76.2 115.57 90)
       (effects (font (size 1.143 1.143)) (justify left))
@@
   )
   (symbol (lib_id "LRJ-parts:C_CL21B105KBFNNNF") (at 73.66 111.76 90) (unit 1)
-    (in_bom yes) (on_board yes)
+    (in_bom no) (on_board no)
     (property "Reference" "C26" (id 0) (at 74.93 110.49 90)
       (effects (font (size 1.143 1.143)))
@@
   )
   (symbol (lib_id "LRJ-parts:C_CC0805JPX7R9BB104") (at 64.77 105.41 90) (unit 1)
-    (in_bom yes) (on_board yes)
+    (in_bom no) (on_board no)
     (property "Reference" "C11" (id 0) (at 63.5 104.14 90)
       (effects (font (size 1.143 1.143)) (justify left))
@@
       (reference "#PWR0120") (unit 1) (value "GND") (footprint "")
     )
+    (path "/d5c7e94e-ee8c-4fa2-b6f9-333fadc34caa/257766af-5a69-4b0b-9011-86f530c64d0b"
+      (reference "#PWR0121") (unit 1) (value "+5V") (footprint "")
+    )
     (path "/bc7b9d52-219c-453a-9752-d4491f369786/17275835-3b83-40ba-9db4-48a2a603bad3"
       (reference "#PWR0122") (unit 1) (value "+5V") (footprint "")
@@
     )
     (path "/d5c7e94e-ee8c-4fa2-b6f9-333fadc34caa/8a4185ef-ebab-4be1-9b5b-f382187c169e"
-      (reference "X1") (unit 1) (value "14.31818MHz ") (footprint "Oscillator:Oscillator_DIP-14")
+      (reference "X1") (unit 1) (value "14.31818MHz ") (footprint "Oscillator:Oscillator_DIP-8")
     )
     (path "/d5c7e94e-ee8c-4fa2-b6f9-333fadc34caa/6f712bc1-4eb0-439a-a5fd-bb1c6396a84d"

Commit message: Updates during tests with prototype
Connections:
- net ~{BUSDIR}: now also U7.11 (4Y)
- net ~{RD}: now also U7.13 (4B)
- net at U7.12 (4A): now also U4.9 (~{Y6}), U7.2 (1B), U7.5 (2B)
- no-connect marks 11 -> 8
Changed lines of the file:
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@@
     (title "TRH9000")
     (date "2022-08-04")
-    (rev "0")
+    (rev "1")
     (company "The Retro Hacker")
     (comment 2 "Shared under CERN-OHL-S license")
@@
     (comment 4 "Designed  by: Cristiano Goncalves")
   )
+  (junction (at 234.95 82.55) (diameter 0) (color 0 0 0 0)
+  )
   (junction (at 144.78 113.03) (diameter 0) (color 0 0 0 0)
   )
@@
   )
   (junction (at 80.01 116.84) (diameter 0) (color 0 0 0 0)
+  )
+  (junction (at 238.76 97.79) (diameter 0) (color 0 0 0 0)
   )
   (junction (at 137.16 105.41) (diameter 0) (color 0 0 0 0)
@@
   (no_connect (at 224.79 95.25))
   (no_connect (at 224.79 87.63))
-  (no_connect (at 247.65 100.33))
-  (no_connect (at 247.65 97.79))
-  (no_connect (at 267.97 100.33))
   (no_connect (at 118.11 107.95))
   (bus_entry (at 160.02 77.47) (size -2.54 2.54)
@@
     (stroke (width 0) (type default) (color 0 0 0 0))
   )
+  (wire (pts (xy 238.76 97.79) (xy 247.65 97.79))
+    (stroke (width 0) (type default) (color 0 0 0 0))
+  )
   (wire (pts (xy 201.93 99.06) (xy 205.74 99.06))
     (stroke (width 0) (type default) (color 0 0 0 0))
   )
-  (wire (pts (xy 242.57 107.95) (xy 242.57 95.25))
-    (stroke (width 0) (type default) (color 0 0 0 0))
-  )
   (bus (pts (xy 160.02 77.47) (xy 160.02 80.01))
     (stroke (width 0) (type default) (color 0 0 0 0))
@@
     (stroke (width 0) (type default) (color 0 0 0 0))
   )
+  (wire (pts (xy 234.95 100.33) (xy 247.65 100.33))
+    (stroke (width 0) (type default) (color 0 0 0 0))
+  )
+  (wire (pts (xy 242.57 95.25) (xy 242.57 113.03))
+    (stroke (width 0) (type default) (color 0 0 0 0))
+  )
   (wire (pts (xy 118.11 49.53) (xy 123.19 49.53))
     (stroke (width 0) (type default) (color 0 0 0 0))
@@
     (stroke (width 0) (type default) (color 0 0 0 0))
   )
+  (wire (pts (xy 267.97 100.33) (xy 274.32 100.33))
+    (stroke (width 0) (type default) (color 0 0 0 0))
+  )
   (wire (pts (xy 82.55 52.07) (xy 87.63 52.07))
     (stroke (width 0) (type default) (color 0 0 0 0))
@@
     (stroke (width 0) (type default) (color 0 0 0 0))
   )
+  (wire (pts (xy 234.95 82.55) (xy 247.65 82.55))
+    (stroke (width 0) (type default) (color 0 0 0 0))
+  )
   (wire (pts (xy 76.2 111.76) (xy 80.01 111.76))
     (stroke (width 0) (type default) (color 0 0 0 0))
@@
     (stroke (width 0) (type default) (color 0 0 0 0))
   )
+  (wire (pts (xy 234.95 100.33) (xy 234.95 82.55))
+    (stroke (width 0) (type default) (color 0 0 0 0))
+  )
   (wire (pts (xy 118.11 46.99) (xy 123.19 46.99))
     (stroke (width 0) (type default) (color 0 0 0 0))
@@
     (stroke (width 0) (type default) (color 0 0 0 0))
   )
-  (wire (pts (xy 243.84 82.55) (xy 247.65 82.55))
+  (wire (pts (xy 232.41 82.55) (xy 234.95 82.55))
     (stroke (width 0) (type default) (color 0 0 0 0))
   )
@@
     (stroke (width 0) (type default) (color 0 0 0 0))
   )
-  (wire (pts (xy 238.76 107.95) (xy 242.57 107.95))
+  (wire (pts (xy 213.36 113.03) (xy 242.57 113.03))
     (stroke (width 0) (type default) (color 0 0 0 0))
   )
@@
   )
   (text "The MSX system-clock\nis often set to 3.58MHz -\naka, the same as the\nsub-carrier clock of NTSC."
-    (at 231.14 120.65 0)
+    (at 207.01 127 0)
     (effects (font (size 1.524 1.524)) (justify left bottom))
   )
@@
     (effects (font (size 1.27 1.27)) (justify left bottom))
   )
+  (label "~{BUSDIR}" (at 274.32 100.33 0)
+    (effects (font (size 1.524 1.524)) (justify left bottom))
+  )
   (label "~{RD}" (at 81.28 62.23 180)
     (effects (font (size 1.27 1.27)) (justify right bottom))
@@
     (effects (font (size 1.27 1.27)) (justify right bottom))
   )
-  (label "~{RD}" (at 243.84 82.55 180)
+  (label "~{RD}" (at 232.41 82.55 180)
     (effects (font (size 1.27 1.27)) (justify right bottom))
   )
@@
     (effects (font (size 1.27 1.27)) (justify left bottom))
   )
-  (label "SYS_CLK" (at 238.76 107.95 180)
+  (label "SYS_CLK" (at 213.36 113.03 180)
     (effects (font (size 1.27 1.27)) (justify right bottom))
   )
@@
     (pin "8")
     (pin "9")
-    (pin "14")
-    (pin "7")
   )
   (symbol (lib_id "LRJ-parts:C_CL21B105KBFNNNF") (at 142.24 113.03 90) (unit 1)
@@
     (pin "7")
     (pin "9")
-    (pin "16")
-    (pin "8")
   )
   (symbol (lib_id "power:+5V") (at 137.16 36.83 0) (unit 1)

Commit message: Multiple changes. Check the dev log.
Parts:
- removed C11, C12: 0.1uF, Capacitor_SMD:C_0805_2012Metric, symbol LRJ-parts:C_CC0805JPX7R9BB104
- removed C25, C26: 1 µF, Capacitor_SMD:C_0805_2012Metric, symbol LRJ-parts:C_CL21B105KBFNNNF
- renumbered C10 to C1, C27 to C2, U4 to U1, U7 to U2
Connections:
- net +12V: no longer names the net of BUS1.48 (+12V)
- net -12V: no longer names the net of BUS1.50 (-12V)
- no-connect marks 8 -> 10

Commit message: Multiple changes.
Parts:
- removed Cart1: MSX-cartridge_dummy, trh9000:MSX-cart-dummy, symbol TRH9000:MSX-cartridge_dummy
Connections:
- net SCIN is gone; now on net ~{BUSDIR}: U2.8 (3Y)
- net A3: now also U1.1 (A0)
- net A4: now also U1.4 (~{G2A}); no longer U1.1 (A0)
- net SYS_CLK: no longer U2.10 (3B), U2.9 (3A)
- net VDP/~{VDPR}: now also U2.11 (4Y); no longer U2.3 (1Y)
- net VDP/~{VDPW}: now also U2.3 (1Y); no longer U2.6 (2Y)
- net ~{BUSDIR}: no longer U2.11 (4Y)
- net ~{IORQ}: now also U2.5 (2B); no longer U1.4 (~{G2A})
- net ~{RD}: now also U2.9 (3A); no longer U2.1 (1A)
- net ~{WR}: now also U2.2 (1B); no longer U2.4 (2A)
- new net: U2.1 (1A), U2.10 (3B), U2.12 (4A), U2.6 (2Y)
- new net: U1.9 (~{Y6}), U2.4 (2A)
Other:
- sheet VIDEO ports: added none; removed SCIN
- note removed: "Cartridge-dummy - to allow testing of the mechanical form-factor."
- note removed: "LEGEND: ------ VDP = Video Display Processor CLK = Clock SLTSL = Slot Select signal CS = Chip Select SYS_CLK = MSX System Clock"
- note removed: "The MSX system-clock is often set to 3.58MHz - aka, the same as the sub-carrier clock of NTSC."
- moved on the sheet: BUS1, C1, C2, U1A, U2A

Commit message: Multiple changes.
Parts:
- removed C1: 0.1uF, Capacitor_SMD:C_0805_2012Metric, symbol LRJ-parts:C_CC0805JPX7R9BB104
- removed C2: 1 µF, Capacitor_SMD:C_0805_2012Metric, symbol LRJ-parts:C_CL21B105KBFNNNF
- added C1: 0.1uF, Capacitor_SMD:C_0805_2012Metric, symbol Device:C
- added C2: 10uF, Capacitor_SMD:C_0805_2012Metric, symbol Device:C
Connections:
- net +5V: now also C1.1, C2.1
- net GND: now also C1.2, C2.2
- net ~{MERQ}: no longer names the net of BUS1.12 (~{MERQ})
- no-connect marks 10 -> 11
