File: Hardware/Kicad/TRH9000_1.7/TRH9000.kicad_pcb (KiCad board)
At the start: 4 copper layers, 100 x 77.5 mm, 66 parts, among them J2 RGB, J3 Composite, J4 SVIDEO, Q1 BC817, U1 74HC138, U2 74HC32, U3 V9990, U4 KM428C256, U5 KM428C256, U6 CXA2075M, X1 14.31818MHz, Y1 21.47727Mhz

Commit message: Content organization. README.MD update.
Parts:
- removed TRH1: LOGO, trh9000:TRH
- added G***: LOGO, Footprints:LOGO_TRH_11, F.Cu at (119.6, 114.8)
